File: Pi_Board.kicad_pcb (KiCad board)
At the start: 4 copper layers, 148.9 x 130 mm, 50 parts, among them J1 USBR-A-S-F-O-VU, J10 5-1775444-9, J11 BM04B-ACHSS-GAN-TF, J2 1-2199230-5, J3 10029449-111RLF, J4 DE9_Plug, J5 J0011D01BNL, J6 Conn_01x02_Socket, J7 104031-0811, J8 10029449-111RLF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

Commit message: pushed V1
Parts:
- added G***: LOGO, LOGO, B.Cu at (135.2, 90.1)
- J7: value 104031-0811 -> SDCARD_MOLEX_503398-1892
Routing:
- net GND: track 226.0 -> 231.9 mm
- net /3V3: track 385.0 -> 382.8 mm
- net /I2C_SCL: track 170.5 -> 169.9 mm
- net /SD_DAT2: track 145.6 -> 146.1 mm
Other:
- board text added: "PI MINI V1"
- board text added: "https://github.com/brendena/mini_pi"
